File: keyboard.kicad_sch (KiCad schematic)
At the start: 12 parts, among them U1 Teensy4.1, U101 CAT24C256, U102 AP22653AW6-7

Commit message: Fleshed out layout
Parts:
- removed C102: 10u, Capacitor_SMD:C_0603_1608Metric, symbol Device:C
- removed C103, C104: 0.1u, Capacitor_SMD:C_0603_1608Metric, symbol Device:C
- removed C105: 120u, Capacitor_SMD:C_0603_1608Metric, symbol Device:C
- removed R103: 10k, Resistor_SMD:R_0603_1608Metric, symbol Device:R_US
- removed R104: 50k, Resistor_SMD:R_0603_1608Metric, symbol Device:R_US
- removed U101: CAT24C256, Package_SO:TSSOP-8_4.4x3mm_P0.65mm, symbol Memory_EEPROM:CAT24C256
- removed U102: AP22653AW6-7, Package_TO_SOT_SMD:SOT-23-6_Handsoldering, symbol Keyboard:AP22653AW6-7
- added U102: CAT24C256, Package_SO:TSSOP-8_4.4x3mm_P0.65mm, symbol Memory_EEPROM:CAT24C256
- C101: footprint Capacitor_SMD:C_0603_1608Metric -> Capacitor_SMD:C_0805_2012Metric
- R101, R102: footprint Resistor_SMD:R_0603_1608Metric -> Resistor_SMD:R_0805_2012Metric
- U101: renamed from U1; footprint Teensy:Teensy41 -> Keyboard:Teensy41; symbol teensy:Teensy4.1 -> Keyboard:Teensy4.1
Connections:
- net VBUS is gone; now on net +5V: U101.49 (VUSB)
- net +3V3: now also U102.8 (VCC)
- net GND: now also U102.1 (A0), U102.2 (A1), U102.3 (A2), U102.4 (GND), U102.7 (WP); no longer U101.52 (GND), U101.58 (GND), U101.59 (GND)
- net SCL: now also U102.6 (SCL)
- net SDA: now also U102.5 (SDA)
- net EN renamed VSYNC
- net ~{FAULT} renamed VIO_EN
Other:
- sheet Keyboard Matrix ports: added CS[0..99], SW[0..21]; removed ledh[0..103], ledl[0..103]
- sheet LED Drive ports: added CS[0..99], SCL, SDA, SW[0..21], VIO_EN, VSYNC; removed EN, ledh[0..103], ledl[0..103], ~{FAULT}
