File: keyboard_matrix.kicad_sch (KiCad schematic)
At the start: 312 parts, among them SW2000 MX-LED, SW2001 MX-LED, SW2002 F2, SW2003 F3, SW2004 F4, SW2005 F5, SW2006 F6, SW2007 F7, SW2008 F8, SW2009 F9, SW2010 F10, SW2011 F11, SW2012 F12, SW2013 PrtSc, SW2014 ScrLk, SW2015 Pause, SW2017 1, SW2018 2, SW2019 3, SW2020 4, SW2021 5, SW2022 6, SW2023 7, SW2024 8, SW2025 9, SW2026 0, SW2027 -, SW2028 =, SW2029 Bksp, SW2030 Ins, SW2031 Home, SW2032 PgUp, SW2033 NumLk, SW2034 /, SW2035 *, SW2036 -, SW2037 Tab, SW2038 Q, SW2039 W, SW2040 E, SW2041 R, SW2042 T, SW2043 Y, SW2044 U, SW2045 I, SW2046 O, SW2047 P, SW2048 [, SW2049 ], SW2050 \, SW2051 Del, SW2052 End, SW2053 PgDn, SW2054 7, SW2055 8, SW2056 9, SW2057 +, SW2058 Caps Lock, SW2059 A, SW2060 S, SW2061 D, SW2062 F, SW2063 G, SW2064 H, SW2065 J, SW2066 K, SW2067 L, SW2068 ;, SW2069 ', SW2070 Enter, SW2071 4, SW2072 5, SW2073 6, SW2074 Shift, SW2075 Z, SW2076 X, SW2077 C, SW2078 V, SW2079 B, SW2080 N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

Commit message: Fleshed out layout
Parts:
- SW2000: renamed from SW2104; value MX-LED -> Esc; footprint (none) -> Keyboard:MXOnly-1U-Hotswap
- SW2000: value MX-LED -> Esc; footprint (none) -> Keyboard:MXOnly-1U-Hotswap
- SW2001: renamed from SW2105; value MX-LED -> F1; footprint (none) -> Keyboard:MXOnly-1U-Hotswap
- SW2001: value MX-LED -> F1; footprint (none) -> Keyboard:MXOnly-1U-Hotswap
- SW2002: renamed from SW2106; value MX-LED -> F2; footprint (none) -> Keyboard:MXOnly-1U-Hotswap
- SW2003: renamed from SW2107; value MX-LED -> F3; footprint (none) -> Keyboard:MXOnly-1U-Hotswap
- SW2004: renamed from SW2108; value MX-LED -> F4; footprint (none) -> Keyboard:MXOnly-1U-Hotswap
- SW2005: renamed from SW2109; value MX-LED -> F5; footprint (none) -> Keyboard:MXOnly-1U-Hotswap
- SW2006: renamed from SW2110; value MX-LED -> F6; footprint (none) -> Keyboard:MXOnly-1U-Hotswap
- SW2007: renamed from SW2111; value MX-LED -> F7; footprint (none) -> Keyboard:MXOnly-1U-Hotswap
- SW2008: renamed from SW2112; value MX-LED -> F8; footprint (none) -> Keyboard:MXOnly-1U-Hotswap
- SW2009: renamed from SW2113; value MX-LED -> F9; footprint (none) -> Keyboard:MXOnly-1U-Hotswap
- SW2010: renamed from SW2114; value MX-LED -> F10; footprint (none) -> Keyboard:MXOnly-1U-Hotswap
- SW2011: renamed from SW2115; value MX-LED -> F11; footprint (none) -> Keyboard:MXOnly-1U-Hotswap
- SW2012: renamed from SW2116; value MX-LED -> F12; footprint (none) -> Keyboard:MXOnly-1U-Hotswap
- SW2013: renamed from SW2117; value MX-LED -> PrtSc; footprint (none) -> Keyboard:MXOnly-1U-Hotswap
- SW2014: renamed from SW2118; value MX-LED -> ScrLk; footprint (none) -> Keyboard:MXOnly-1U-Hotswap
- SW2015: renamed from SW2119; value MX-LED -> Pause; footprint (none) -> Keyboard:MXOnly-1U-Hotswap
- SW2016: renamed from SW2120; value MX-LED -> `; footprint (none) -> Keyboard:MXOnly-1U-Hotswap
- SW2016: value ~ -> `
- SW2017: renamed from SW2121; value MX-LED -> 1; footprint (none) -> Keyboard:MXOnly-1U-Hotswap
- SW2018: renamed from SW2122; value MX-LED -> 2; footprint (none) -> Keyboard:MXOnly-1U-Hotswap
- SW2019: renamed from SW2123; value MX-LED -> 3; footprint (none) -> Keyboard:MXOnly-1U-Hotswap
- SW2020: renamed from SW2124; value MX-LED -> 4; footprint (none) -> Keyboard:MXOnly-1U-Hotswap
- SW2021: renamed from SW2125; value MX-LED -> 5; footprint (none) -> Keyboard:MXOnly-1U-Hotswap
- SW2022: renamed from SW2126; value MX-LED -> 6; footprint (none) -> Keyboard:MXOnly-1U-Hotswap
- SW2023: renamed from SW2127; value MX-LED -> 7; footprint (none) -> Keyboard:MXOnly-1U-Hotswap
- SW2024: renamed from SW2128; value MX-LED -> 8; footprint (none) -> Keyboard:MXOnly-1U-Hotswap
- SW2025: renamed from SW2129; value MX-LED -> 9; footprint (none) -> Keyboard:MXOnly-1U-Hotswap
- SW2026: renamed from SW2130; value MX-LED -> 0; footprint (none) -> Keyboard:MXOnly-1U-Hotswap
- SW2027: renamed from SW2131; value MX-LED -> -; footprint (none) -> Keyboard:MXOnly-1U-Hotswap
- SW2028: renamed from SW2132; value MX-LED -> =; footprint (none) -> Keyboard:MXOnly-1U-Hotswap
- SW2029: renamed from SW2133; value MX-LED -> Bksp; footprint (none) -> Keyboard:MXOnly-2U-Hotswap
- SW2030: renamed from SW2134; value MX-LED -> Ins; footprint (none) -> Keyboard:MXOnly-1U-Hotswap
- SW2031: renamed from SW2135; value MX-LED -> Home; footprint (none) -> Keyboard:MXOnly-1U-Hotswap
- SW2032: renamed from SW2136; value MX-LED -> PgUp; footprint (none) -> Keyboard:MXOnly-1U-Hotswap
- SW2033: renamed from SW2137; value MX-LED -> NumLk; footprint (none) -> Keyboard:MXOnly-1U-Hotswap
- SW2034: renamed from SW2138; value MX-LED -> /; footprint (none) -> Keyboard:MXOnly-1U-Hotswap
- SW2035: renamed from SW2139; value MX-LED -> *; footprint (none) -> Keyboard:MXOnly-1U-Hotswap
- SW2036: renamed from SW2140; value MX-LED -> -; footprint (none) -> Keyboard:MXOnly-1U-Hotswap
- SW2037: renamed from SW2141; value MX-LED -> Tab; footprint (none) -> Keyboard:MXOnly-1.5U-Hotswap
- SW2038: renamed from SW2142; value MX-LED -> Q; footprint (none) -> Keyboard:MXOnly-1U-Hotswap
- SW2039: renamed from SW2143; value MX-LED -> W; footprint (none) -> Keyboard:MXOnly-1U-Hotswap
- SW2040: renamed from SW2144; value MX-LED -> E; footprint (none) -> Keyboard:MXOnly-1U-Hotswap
- SW2041: renamed from SW2145; value MX-LED -> R; footprint (none) -> Keyboard:MXOnly-1U-Hotswap
- SW2042: renamed from SW2146; value MX-LED -> T; footprint (none) -> Keyboard:MXOnly-1U-Hotswap
- SW2043: renamed from SW2147; value MX-LED -> Y; footprint (none) -> Keyboard:MXOnly-1U-Hotswap
- SW2044: renamed from SW2148; value MX-LED -> U; footprint (none) -> Keyboard:MXOnly-1U-Hotswap
- SW2045: renamed from SW2149; value MX-LED -> I; footprint (none) -> Keyboard:MXOnly-1U-Hotswap
- SW2046: renamed from SW2150; value MX-LED -> O; footprint (none) -> Keyboard:MXOnly-1U-Hotswap
- SW2047: renamed from SW2151; value MX-LED -> P; footprint (none) -> Keyboard:MXOnly-1U-Hotswap
- SW2048: renamed from SW2152; value MX-LED -> [; footprint (none) -> Keyboard:MXOnly-1U-Hotswap
- SW2049: renamed from SW2153; value MX-LED -> ]; footprint (none) -> Keyboard:MXOnly-1U-Hotswap
- SW2050: renamed from SW2154; value MX-LED -> \; footprint (none) -> Keyboard:MXOnly-1.5U-Hotswap
- SW2051: renamed from SW2155; value MX-LED -> Del; footprint (none) -> Keyboard:MXOnly-1U-Hotswap
- SW2052: renamed from SW2156; value MX-LED -> End; footprint (none) -> Keyboard:MXOnly-1U-Hotswap
- SW2053: renamed from SW2157; value MX-LED -> PgDn; footprint (none) -> Keyboard:MXOnly-1U-Hotswap
- SW2054: renamed from SW2158; value MX-LED -> 7; footprint (none) -> Keyboard:MXOnly-1U-Hotswap
- SW2055: renamed from SW2159; value MX-LED -> 8; footprint (none) -> Keyboard:MXOnly-1U-Hotswap
- SW2056: renamed from SW2160; value MX-LED -> 9; footprint (none) -> Keyboard:MXOnly-1U-Hotswap
- SW2057: renamed from SW2161; value MX-LED -> +; footprint (none) -> Keyboard:MXOnly-2U-Hotswap
- SW2058: renamed from SW2162; value MX-LED -> Caps Lock; footprint (none) -> Keyboard:MXOnly-1.75U-Hotswap
- SW2059: renamed from SW2163; value MX-LED -> A; footprint (none) -> Keyboard:MXOnly-1U-Hotswap
- SW2060: renamed from SW2164; value MX-LED -> S; footprint (none) -> Keyboard:MXOnly-1U-Hotswap
- SW2061: renamed from SW2165; value MX-LED -> D; footprint (none) -> Keyboard:MXOnly-1U-Hotswap
- SW2062: renamed from SW2166; value MX-LED -> F; footprint (none) -> Keyboard:MXOnly-1U-Hotswap
- SW2063: renamed from SW2167; value MX-LED -> G; footprint (none) -> Keyboard:MXOnly-1U-Hotswap
- SW2064: renamed from SW2168; value MX-LED -> H; footprint (none) -> Keyboard:MXOnly-1U-Hotswap
- SW2065: renamed from SW2169; value MX-LED -> J; footprint (none) -> Keyboard:MXOnly-1U-Hotswap
- SW2066: renamed from SW2170; value MX-LED -> K; footprint (none) -> Keyboard:MXOnly-1U-Hotswap
- SW2067: renamed from SW2171; value MX-LED -> L; footprint (none) -> Keyboard:MXOnly-1U-Hotswap
- SW2068: renamed from SW2172; value MX-LED -> ;; footprint (none) -> Keyboard:MXOnly-1U-Hotswap
- SW2069: renamed from SW2173; value MX-LED -> '; footprint (none) -> Keyboard:MXOnly-1U-Hotswap
- SW2070: renamed from SW2174; value MX-LED -> Enter; footprint (none) -> Keyboard:MXOnly-2.25U-Hotswap
- SW2071: renamed from SW2175; value MX-LED -> 4; footprint (none) -> Keyboard:MXOnly-1U-Hotswap
- SW2072: renamed from SW2176; value MX-LED -> 5; footprint (none) -> Keyboard:MXOnly-1U-Hotswap
- SW2073: renamed from SW2177; value MX-LED -> 6; footprint (none) -> Keyboard:MXOnly-1U-Hotswap
- SW2074: renamed from SW2178; value MX-LED -> Shift; footprint (none) -> Keyboard:MXOnly-2.25U-Hotswap
- SW2075: renamed from SW2179; value MX-LED -> Z; footprint (none) -> Keyboard:MXOnly-1U-Hotswap
- SW2076: renamed from SW2180; value MX-LED -> X; footprint (none) -> Keyboard:MXOnly-1U-Hotswap
- SW2077: renamed from SW2181; value MX-LED -> C; footprint (none) -> Keyboard:MXOnly-1U-Hotswap
- SW2078: renamed from SW2182; value MX-LED -> V; footprint (none) -> Keyboard:MXOnly-1U-Hotswap
- SW2079: renamed from SW2183; value MX-LED -> B; footprint (none) -> Keyboard:MXOnly-1U-Hotswap
- SW2080: renamed from SW2184; value MX-LED -> N; footprint (none) -> Keyboard:MXOnly-1U-Hotswap
- SW2081: renamed from SW2185; value MX-LED -> M; footprint (none) -> Keyboard:MXOnly-1U-Hotswap
- SW2082: renamed from SW2186; value MX-LED -> ,; footprint (none) -> Keyboard:MXOnly-1U-Hotswap
- SW2083: renamed from SW2187; value MX-LED -> .; footprint (none) -> Keyboard:MXOnly-1U-Hotswap
- SW2084: renamed from SW2188; value MX-LED -> /; footprint (none) -> Keyboard:MXOnly-1U-Hotswap
- SW2085: renamed from SW2189; value MX-LED -> Shift; footprint (none) -> Keyboard:MXOnly-2.75U-Hotswap
- SW2086: renamed from SW2190; value MX-LED -> Up; footprint (none) -> Keyboard:MXOnly-1U-Hotswap
- SW2087: renamed from SW2191; value MX-LED -> 1; footprint (none) -> Keyboard:MXOnly-1U-Hotswap
- SW2088: renamed from SW2192; value MX-LED -> 2; footprint (none) -> Keyboard:MXOnly-1U-Hotswap
- SW2089: renamed from SW2193; value MX-LED -> 3; footprint (none) -> Keyboard:MXOnly-1U-Hotswap
- SW2090: renamed from SW2194; value MX-LED -> Enter; footprint (none) -> Keyboard:MXOnly-2U-Hotswap
- SW2091, SW2092, SW2093, SW2095, SW2096, SW2097, SW2098: footprint Keyboard:MXOnly-1.25U-Hotswap -> Keyboard:MXOnly-1U-Hotswap
- SW2091: renamed from SW2195; value MX-LED -> LCtrl; footprint (none) -> Keyboard:MXOnly-1U-Hotswap
- SW2092: renamed from SW2196; value MX-LED -> Super; footprint (none) -> Keyboard:MXOnly-1U-Hotswap
- SW2093: renamed from SW2197; value MX-LED -> LAlt; footprint (none) -> Keyboard:MXOnly-1U-Hotswap
- SW2094: renamed from SW2198; value MX-LED -> Space; footprint (none) -> Keyboard:MXOnly-6.25U-Hotswap
- SW2095: renamed from SW2199; value MX-LED -> RAlt; footprint (none) -> Keyboard:MXOnly-1U-Hotswap
- SW2096: renamed from SW2200; value MX-LED -> Fn; footprint (none) -> Keyboard:MXOnly-1U-Hotswap
- SW2097: renamed from SW2201; value MX-LED -> RClick; footprint (none) -> Keyboard:MXOnly-1U-Hotswap
- SW2098: renamed from SW2202; value MX-LED -> RCtrl; footprint (none) -> Keyboard:MXOnly-1U-Hotswap
- SW2099: renamed from SW2203; value MX-LED -> Left; footprint (none) -> Keyboard:MXOnly-1U-Hotswap
- SW2100: renamed from SW2204; value MX-LED -> Down; footprint (none) -> Keyboard:MXOnly-1U-Hotswap
- SW2101: renamed from SW2205; value MX-LED -> Right; footprint (none) -> Keyboard:MXOnly-1U-Hotswap
- SW2102: footprint Keyboard:MXOnly-2U-Hotswap -> Keyboard:MXOnly-1U-Hotswap
- SW2102: renamed from SW2206; value MX-LED -> 0; footprint (none) -> Keyboard:MXOnly-1U-Hotswap
- SW2103: renamed from SW2207; value MX-LED -> .; footprint (none) -> Keyboard:MXOnly-1U-Hotswap
Connections:
- net B1 is gone; now on net CS2: SW2001.5 (B)
- net B101 is gone; now on net CS35: SW2101.5 (B)
- net B102 is gone; now on net CS35: SW2102.5 (B)
- net B103 is gone; now on net CS35: SW2103.5 (B)
- net B11 is gone; now on net CS20: SW2011.5 (B)
- net B12 is gone; now on net CS20: SW2012.5 (B)
- net B13 is gone; now on net CS20: SW2013.5 (B)
- net B14 is gone; now on net CS20: SW2014.5 (B)
- net B15 is gone; now on net CS20: SW2015.5 (B)
- net B17 is gone; now on net CS5: SW2017.5 (B)
- net B18 is gone; now on net CS5: SW2018.5 (B)
- net B19 is gone; now on net CS5: SW2019.5 (B)
- net B2 is gone; now on net CS2: SW2002.5 (B)
- net B20 is gone; now on net CS5: SW2020.5 (B)
- net B21 is gone; now on net CS5: SW2021.5 (B)
- net B22 is gone; now on net CS5: SW2022.5 (B)
- net B23 is gone; now on net CS5: SW2023.5 (B)
- net B24 is gone; now on net CS5: SW2024.5 (B)
- net B25 is gone; now on net CS5: SW2025.5 (B)
- net B26 is gone; now on net CS5: SW2026.5 (B)
- net B28 is gone; now on net CS23: SW2028.5 (B)
- net B29 is gone; now on net CS23: SW2029.5 (B)
- net B3 is gone; now on net CS2: SW2003.5 (B)
- net B30 is gone; now on net CS23: SW2030.5 (B)
- net B31 is gone; now on net CS23: SW2031.5 (B)
- net B32 is gone; now on net CS23: SW2032.5 (B)
- net B33 is gone; now on net CS23: SW2033.5 (B)
- net B34 is gone; now on net CS23: SW2034.5 (B)
- net B35 is gone; now on net CS23: SW2035.5 (B)
- net B36 is gone; now on net CS23: SW2036.5 (B)
- net B38 is gone; now on net CS8: SW2038.5 (B)
- net B39 is gone; now on net CS8: SW2039.5 (B)
- net B4 is gone; now on net CS2: SW2004.5 (B)
- net B40 is gone; now on net CS8: SW2040.5 (B)
- net B41 is gone; now on net CS8: SW2041.5 (B)
- net B42 is gone; now on net CS8: SW2042.5 (B)
- net B43 is gone; now on net CS8: SW2043.5 (B)
- net B44 is gone; now on net CS8: SW2044.5 (B)
- net B45 is gone; now on net CS8: SW2045.5 (B)
- net B46 is gone; now on net CS8: SW2046.5 (B)
- net B48 is gone; now on net CS26: SW2048.5 (B)
- net B49 is gone; now on net CS26: SW2049.5 (B)
- net B5 is gone; now on net CS2: SW2005.5 (B)
- net B50 is gone; now on net CS26: SW2050.5 (B)
- net B51 is gone; now on net CS26: SW2051.5 (B)
- net B52 is gone; now on net CS26: SW2052.5 (B)
- net B53 is gone; now on net CS26: SW2053.5 (B)
- net B54 is gone; now on net CS26: SW2054.5 (B)
- net B55 is gone; now on net CS26: SW2055.5 (B)
- net B56 is gone; now on net CS26: SW2056.5 (B)
- net B57 is gone; now on net CS26: SW2057.5 (B)
- net B59 is gone; now on net CS11: SW2059.5 (B)
- net B6 is gone; now on net CS2: SW2006.5 (B)
- net B60 is gone; now on net CS11: SW2060.5 (B)
- net B61 is gone; now on net CS11: SW2061.5 (B)
- net B62 is gone; now on net CS11: SW2062.5 (B)
- net B63 is gone; now on net CS11: SW2063.5 (B)
- net B64 is gone; now on net CS11: SW2064.5 (B)
- net B65 is gone; now on net CS11: SW2065.5 (B)
- net B66 is gone; now on net CS11: SW2066.5 (B)
- net B67 is gone; now on net CS11: SW2067.5 (B)
- net B69 is gone; now on net CS29: SW2069.5 (B)
- net B7 is gone; now on net CS2: SW2007.5 (B)
- net B70 is gone; now on net CS29: SW2070.5 (B)
- net B71 is gone; now on net CS29: SW2071.5 (B)
- net B72 is gone; now on net CS29: SW2072.5 (B)
- net B73 is gone; now on net CS29: SW2073.5 (B)
- net B75 is gone; now on net CS14: SW2075.5 (B)
- net B76 is gone; now on net CS14: SW2076.5 (B)
- net B77 is gone; now on net CS14: SW2077.5 (B)
- net B78 is gone; now on net CS14: SW2078.5 (B)
- net B79 is gone; now on net CS14: SW2079.5 (B)
- net B8 is gone; now on net CS2: SW2008.5 (B)
- net B80 is gone; now on net CS14: SW2080.5 (B)
- net B81 is gone; now on net CS14: SW2081.5 (B)
- net B82 is gone; now on net CS14: SW2082.5 (B)
- net B83 is gone; now on net CS14: SW2083.5 (B)
- net B85 is gone; now on net CS32: SW2085.5 (B)
- net B86 is gone; now on net CS32: SW2086.5 (B)
- net B87 is gone; now on net CS32: SW2087.5 (B)
- net B88 is gone; now on net CS32: SW2088.5 (B)
- net B89 is gone; now on net CS32: SW2089.5 (B)
- net B9 is gone; now on net CS20: SW2009.5 (B)
- net B90 is gone; now on net CS32: SW2090.5 (B)
- net B92 is gone; now on net CS17: SW2092.5 (B)
- net B93 is gone; now on net CS17: SW2093.5 (B)
- net B94 is gone; now on net CS17: SW2094.5 (B)
- net B95 is gone; now on net CS17: SW2095.5 (B)
- net B96 is gone; now on net CS35: SW2096.5 (B)
- net B97 is gone; now on net CS35: SW2097.5 (B)
- net B98 is gone; now on net CS35: SW2098.5 (B)
- net B99 is gone; now on net CS35: SW2099.5 (B)
- net G1 is gone; now on net CS1: SW2001.4 (G)
- net G101 is gone; now on net CS34: SW2101.4 (G)
- net G102 is gone; now on net CS34: SW2102.4 (G)
- net G103 is gone; now on net CS34: SW2103.4 (G)
- net G11 is gone; now on net CS19: SW2011.4 (G)
- net G12 is gone; now on net CS19: SW2012.4 (G)
- net G13 is gone; now on net CS19: SW2013.4 (G)
- net G14 is gone; now on net CS19: SW2014.4 (G)
- net G15 is gone; now on net CS19: SW2015.4 (G)
- net G17 is gone; now on net CS4: SW2017.4 (G)
- net G18 is gone; now on net CS4: SW2018.4 (G)
- net G19 is gone; now on net CS4: SW2019.4 (G)
- net G2 is gone; now on net CS1: SW2002.4 (G)
- net G20 is gone; now on net CS4: SW2020.4 (G)
- net G21 is gone; now on net CS4: SW2021.4 (G)
- net G22 is gone; now on net CS4: SW2022.4 (G)
- net G23 is gone; now on net CS4: SW2023.4 (G)
- net G24 is gone; now on net CS4: SW2024.4 (G)
- net G25 is gone; now on net CS4: SW2025.4 (G)
- net G26 is gone; now on net CS4: SW2026.4 (G)
- net G28 is gone; now on net CS22: SW2028.4 (G)
- net G29 is gone; now on net CS22: SW2029.4 (G)
- net G3 is gone; now on net CS1: SW2003.4 (G)
- net G30 is gone; now on net CS22: SW2030.4 (G)
- net G31 is gone; now on net CS22: SW2031.4 (G)
- net G32 is gone; now on net CS22: SW2032.4 (G)
- net G33 is gone; now on net CS22: SW2033.4 (G)
- net G34 is gone; now on net CS22: SW2034.4 (G)
- net G35 is gone; now on net CS22: SW2035.4 (G)
- net G36 is gone; now on net CS22: SW2036.4 (G)
- net G38 is gone; now on net CS7: SW2038.4 (G)
- net G39 is gone; now on net CS7: SW2039.4 (G)
- net G4 is gone; now on net CS1: SW2004.4 (G)
- net G40 is gone; now on net CS7: SW2040.4 (G)
- net G41 is gone; now on net CS7: SW2041.4 (G)
- net G42 is gone; now on net CS7: SW2042.4 (G)
- net G43 is gone; now on net CS7: SW2043.4 (G)
- net G44 is gone; now on net CS7: SW2044.4 (G)
- net G45 is gone; now on net CS7: SW2045.4 (G)
- net G46 is gone; now on net CS7: SW2046.4 (G)
- net G48 is gone; now on net CS25: SW2048.4 (G)
- net G49 is gone; now on net CS25: SW2049.4 (G)
- net G5 is gone; now on net CS1: SW2005.4 (G)
- net G50 is gone; now on net CS25: SW2050.4 (G)
- net G51 is gone; now on net CS25: SW2051.4 (G)
- net G52 is gone; now on net CS25: SW2052.4 (G)
- net G53 is gone; now on net CS25: SW2053.4 (G)
- net G54 is gone; now on net CS25: SW2054.4 (G)
- net G55 is gone; now on net CS25: SW2055.4 (G)
- net G56 is gone; now on net CS25: SW2056.4 (G)
- net G57 is gone; now on net CS25: SW2057.4 (G)
- net G59 is gone; now on net CS10: SW2059.4 (G)
- net G6 is gone; now on net CS1: SW2006.4 (G)
- net G60 is gone; now on net CS10: SW2060.4 (G)
- net G61 is gone; now on net CS10: SW2061.4 (G)
- net G62 is gone; now on net CS10: SW2062.4 (G)
- net G63 is gone; now on net CS10: SW2063.4 (G)
- net G64 is gone; now on net CS10: SW2064.4 (G)
- net G65 is gone; now on net CS10: SW2065.4 (G)
- net G66 is gone; now on net CS10: SW2066.4 (G)
- net G67 is gone; now on net CS10: SW2067.4 (G)
- net G69 is gone; now on net CS28: SW2069.4 (G)
- net G7 is gone; now on net CS1: SW2007.4 (G)
- net G70 is gone; now on net CS28: SW2070.4 (G)
- net G71 is gone; now on net CS28: SW2071.4 (G)
- net G72 is gone; now on net CS28: SW2072.4 (G)
- net G73 is gone; now on net CS28: SW2073.4 (G)
- net G75 is gone; now on net CS13: SW2075.4 (G)
- net G76 is gone; now on net CS13: SW2076.4 (G)
- net G77 is gone; now on net CS13: SW2077.4 (G)
- net G78 is gone; now on net CS13: SW2078.4 (G)
- net G79 is gone; now on net CS13: SW2079.4 (G)
- net G8 is gone; now on net CS1: SW2008.4 (G)
- net G80 is gone; now on net CS13: SW2080.4 (G)
- net G81 is gone; now on net CS13: SW2081.4 (G)
- net G82 is gone; now on net CS13: SW2082.4 (G)
- net G83 is gone; now on net CS13: SW2083.4 (G)
- net G85 is gone; now on net CS31: SW2085.4 (G)
- net G86 is gone; now on net CS31: SW2086.4 (G)
- net G87 is gone; now on net CS31: SW2087.4 (G)
- net G88 is gone; now on net CS31: SW2088.4 (G)
- net G89 is gone; now on net CS31: SW2089.4 (G)
- net G9 is gone; now on net CS19: SW2009.4 (G)
- net G90 is gone; now on net CS31: SW2090.4 (G)
- net G92 is gone; now on net CS16: SW2092.4 (G)
- net G93 is gone; now on net CS16: SW2093.4 (G)
- net G94 is gone; now on net CS16: SW2094.4 (G)
- net G95 is gone; now on net CS16: SW2095.4 (G)
- net G96 is gone; now on net CS34: SW2096.4 (G)
- net G97 is gone; now on net CS34: SW2097.4 (G)
- net G98 is gone; now on net CS34: SW2098.4 (G)
- net G99 is gone; now on net CS34: SW2099.4 (G)
- net R1 is gone; now on net CS0: SW2001.3 (R)
- net R101 is gone; now on net CS33: SW2101.3 (R)
- net R102 is gone; now on net CS33: SW2102.3 (R)
- net R103 is gone; now on net CS33: SW2103.3 (R)
- net R11 is gone; now on net CS18: SW2011.3 (R)
- net R12 is gone; now on net CS18: SW2012.3 (R)
- net R13 is gone; now on net CS18: SW2013.3 (R)
- net R14 is gone; now on net CS18: SW2014.3 (R)
- net R15 is gone; now on net CS18: SW2015.3 (R)
- net R17 is gone; now on net CS3: SW2017.3 (R)
- net R18 is gone; now on net CS3: SW2018.3 (R)
- net R19 is gone; now on net CS3: SW2019.3 (R)
- net R2 is gone; now on net CS0: SW2002.3 (R)
- net R20 is gone; now on net CS3: SW2020.3 (R)
- net R21 is gone; now on net CS3: SW2021.3 (R)
- net R22 is gone; now on net CS3: SW2022.3 (R)
- net R23 is gone; now on net CS3: SW2023.3 (R)
- net R24 is gone; now on net CS3: SW2024.3 (R)
- net R25 is gone; now on net CS3: SW2025.3 (R)
- net R26 is gone; now on net CS3: SW2026.3 (R)
- net R28 is gone; now on net CS21: SW2028.3 (R)
- net R29 is gone; now on net CS21: SW2029.3 (R)
- net R3 is gone; now on net CS0: SW2003.3 (R)
- net R30 is gone; now on net CS21: SW2030.3 (R)
- net R31 is gone; now on net CS21: SW2031.3 (R)
- net R32 is gone; now on net CS21: SW2032.3 (R)
- net R33 is gone; now on net CS21: SW2033.3 (R)
- net R34 is gone; now on net CS21: SW2034.3 (R)
- net R35 is gone; now on net CS21: SW2035.3 (R)
- net R36 is gone; now on net CS21: SW2036.3 (R)
- net R38 is gone; now on net CS6: SW2038.3 (R)
- net R39 is gone; now on net CS6: SW2039.3 (R)
- net R4 is gone; now on net CS0: SW2004.3 (R)
- net R40 is gone; now on net CS6: SW2040.3 (R)
- net R41 is gone; now on net CS6: SW2041.3 (R)
- net R42 is gone; now on net CS6: SW2042.3 (R)
- net R43 is gone; now on net CS6: SW2043.3 (R)
- net R44 is gone; now on net CS6: SW2044.3 (R)
- net R45 is gone; now on net CS6: SW2045.3 (R)
- net R46 is gone; now on net CS6: SW2046.3 (R)
- net R48 is gone; now on net CS24: SW2048.3 (R)
- net R49 is gone; now on net CS24: SW2049.3 (R)
- net R5 is gone; now on net CS0: SW2005.3 (R)
- net R50 is gone; now on net CS24: SW2050.3 (R)
- net R51 is gone; now on net CS24: SW2051.3 (R)
- net R52 is gone; now on net CS24: SW2052.3 (R)
- net R53 is gone; now on net CS24: SW2053.3 (R)
- net R54 is gone; now on net CS24: SW2054.3 (R)
- net R55 is gone; now on net CS24: SW2055.3 (R)
- net R56 is gone; now on net CS24: SW2056.3 (R)
- net R57 is gone; now on net CS24: SW2057.3 (R)
- net R59 is gone; now on net CS9: SW2059.3 (R)
- net R6 is gone; now on net CS0: SW2006.3 (R)
- net R60 is gone; now on net CS9: SW2060.3 (R)
- net R61 is gone; now on net CS9: SW2061.3 (R)
- net R62 is gone; now on net CS9: SW2062.3 (R)
- net R63 is gone; now on net CS9: SW2063.3 (R)
- net R64 is gone; now on net CS9: SW2064.3 (R)
- net R65 is gone; now on net CS9: SW2065.3 (R)
- net R66 is gone; now on net CS9: SW2066.3 (R)
- net R67 is gone; now on net CS9: SW2067.3 (R)
- net R69 is gone; now on net CS27: SW2069.3 (R)
- net R7 is gone; now on net CS0: SW2007.3 (R)
- net R70 is gone; now on net CS27: SW2070.3 (R)
- net R71 is gone; now on net CS27: SW2071.3 (R)
- net R72 is gone; now on net CS27: SW2072.3 (R)
- net R73 is gone; now on net CS27: SW2073.3 (R)
- net R75 is gone; now on net CS12: SW2075.3 (R)
- net R76 is gone; now on net CS12: SW2076.3 (R)
- net R77 is gone; now on net CS12: SW2077.3 (R)
- net R78 is gone; now on net CS12: SW2078.3 (R)
- net R79 is gone; now on net CS12: SW2079.3 (R)
- net R8 is gone; now on net CS0: SW2008.3 (R)
- net R80 is gone; now on net CS12: SW2080.3 (R)
- net R81 is gone; now on net CS12: SW2081.3 (R)
- net R82 is gone; now on net CS12: SW2082.3 (R)
- net R83 is gone; now on net CS12: SW2083.3 (R)
- net R85 is gone; now on net CS30: SW2085.3 (R)
- net R86 is gone; now on net CS30: SW2086.3 (R)
- net R87 is gone; now on net CS30: SW2087.3 (R)
- net R88 is gone; now on net CS30: SW2088.3 (R)
- net R89 is gone; now on net CS30: SW2089.3 (R)
- net R9 is gone; now on net CS18: SW2009.3 (R)
- net R90 is gone; now on net CS30: SW2090.3 (R)
- net R92 is gone; now on net CS15: SW2092.3 (R)
- net R93 is gone; now on net CS15: SW2093.3 (R)
- net R94 is gone; now on net CS15: SW2094.3 (R)
- net R95 is gone; now on net CS15: SW2095.3 (R)
- net R96 is gone; now on net CS33: SW2096.3 (R)
- net R97 is gone; now on net CS33: SW2097.3 (R)
- net R98 is gone; now on net CS33: SW2098.3 (R)
- net R99 is gone; now on net CS33: SW2099.3 (R)
- net row1: now also D_17.1 (K)
- net row4: now also D_74.1 (K)
- net row5: now also D_92.1 (K)
- net at D_76.2 (A): now also SW2076.2 (ROW)
- net at SW2019.2 (ROW): now also D_19.2 (A)
- net at D_92.2 (A): now also SW2092.2 (ROW)
- net at SW2074.2 (ROW): now also D_74.2 (A)
- net at SW2018.2 (ROW): now also D_18.2 (A)
- net at D_93.2 (A): now also SW2093.2 (ROW)
- net at D_1.2 (A): now also SW2001.2 (ROW)
- net at SW2017.2 (ROW): now also D_17.2 (A)
- net at D_2.2 (A): now also SW2002.2 (ROW)
- net at SW2060.2 (ROW): now also D_60.2 (A)
- net at D_75.2 (A): now also SW2075.2 (ROW)
- net B0 renamed CS2
- net B10 renamed CS20
- net B100 renamed CS35
- net B16 renamed CS5
- net B27 renamed CS23
- net B37 renamed CS8
- net B47 renamed CS26
- net B58 renamed CS11
- net B68 renamed CS29
- net B74 renamed CS14
- net B84 renamed CS32
- net B91 renamed CS17
- removed net COM: SW2000.6 (COM), SW2001.6 (COM), SW2002.6 (COM), SW2003.6 (COM), SW2004.6 (COM), SW2005.6 (COM), SW2006.6 (COM), SW2007.6 (COM), SW2008.6 (COM), SW2009.6 (COM), SW2010.6 (COM), SW2011.6 (COM), SW2012.6 (COM), SW2013.6 (COM), SW2014.6 (COM), SW2015.6 (COM), SW2016.6 (COM), SW2017.6 (COM), SW2018.6 (COM), SW2019.6 (COM), SW2020.6 (COM), SW2021.6 (COM), SW2022.6 (COM), SW2023.6 (COM), SW2024.6 (COM), SW2025.6 (COM), SW2026.6 (COM), SW2027.6 (COM), SW2028.6 (COM), SW2029.6 (COM), SW2030.6 (COM), SW2031.6 (COM), SW2032.6 (COM), SW2033.6 (COM), SW2034.6 (COM), SW2035.6 (COM), SW2036.6 (COM), SW2037.6 (COM), SW2038.6 (COM), SW2039.6 (COM), SW2040.6 (COM), SW2041.6 (COM), SW2042.6 (COM), SW2043.6 (COM), SW2044.6 (COM), SW2045.6 (COM), SW2046.6 (COM), SW2047.6 (COM), SW2048.6 (COM), SW2049.6 (COM), SW2050.6 (COM), SW2051.6 (COM), SW2052.6 (COM), SW2053.6 (COM), SW2054.6 (COM), SW2055.6 (COM), SW2056.6 (COM), SW2057.6 (COM), SW2058.6 (COM), SW2059.6 (COM), SW2060.6 (COM), SW2061.6 (COM), SW2062.6 (COM), SW2063.6 (COM), SW2064.6 (COM), SW2065.6 (COM), SW2066.6 (COM), SW2067.6 (COM), SW2068.6 (COM), SW2069.6 (COM), SW2070.6 (COM), SW2071.6 (COM), SW2072.6 (COM), SW2073.6 (COM), SW2074.6 (COM), SW2075.6 (COM), SW2076.6 (COM), SW2077.6 (COM), SW2078.6 (COM), SW2079.6 (COM), SW2080.6 (COM), SW2081.6 (COM), SW2082.6 (COM), SW2083.6 (COM), SW2084.6 (COM), SW2085.6 (COM), SW2086.6 (COM), SW2087.6 (COM), SW2088.6 (COM), SW2089.6 (COM), SW2090.6 (COM), SW2091.6 (COM), SW2092.6 (COM), SW2093.6 (COM), SW2094.6 (COM), SW2095.6 (COM), SW2096.6 (COM), SW2097.6 (COM), SW2098.6 (COM), SW2099.6 (COM), SW2100.6 (COM), SW2101.6 (COM), SW2102.6 (COM), SW2103.6 (COM)
- net G0 renamed CS1
- net G10 renamed CS19
- net G100 renamed CS34
- net G16 renamed CS4
- net G27 renamed CS22
- net G37 renamed CS7
- net G47 renamed CS25
- net G58 renamed CS10
- net G68 renamed CS28
- net G74 renamed CS13
- net G84 renamed CS31
- net G91 renamed CS16
- net R0 renamed CS0
- net R10 renamed CS18
- net R100 renamed CS33
- net R16 renamed CS3
- net R27 renamed CS21
- net R37 renamed CS6
- net R47 renamed CS24
- net R58 renamed CS9
- net R68 renamed CS27
- net R74 renamed CS12
- net R84 renamed CS30
- net R91 renamed CS15
- new net SW0: SW2000.6 (COM), SW2016.6 (COM), SW2037.6 (COM), SW2058.6 (COM), SW2091.6 (COM)
- new net SW1: SW2017.6 (COM), SW2074.6 (COM), SW2092.6 (COM)
- new net SW10: SW2008.6 (COM), SW2026.6 (COM), SW2046.6 (COM), SW2067.6 (COM), SW2083.6 (COM), SW2095.6 (COM)
- new net SW11: SW2009.6 (COM), SW2027.6 (COM), SW2047.6 (COM), SW2068.6 (COM), SW2084.6 (COM), SW2096.6 (COM)
- new net SW12: SW2010.6 (COM), SW2028.6 (COM), SW2048.6 (COM), SW2069.6 (COM)
- new net SW13: SW2011.6 (COM), SW2049.6 (COM), SW2070.6 (COM), SW2085.6 (COM), SW2097.6 (COM)
- new net SW14: SW2012.6 (COM), SW2029.6 (COM), SW2050.6 (COM), SW2098.6 (COM)
- new net SW15: SW2013.6 (COM), SW2030.6 (COM), SW2051.6 (COM), SW2099.6 (COM)
- new net SW16: SW2014.6 (COM), SW2031.6 (COM), SW2052.6 (COM), SW2086.6 (COM), SW2100.6 (COM)
- new net SW17: SW2015.6 (COM), SW2032.6 (COM), SW2053.6 (COM), SW2101.6 (COM)
- new net SW18: SW2033.6 (COM), SW2054.6 (COM), SW2071.6 (COM), SW2087.6 (COM), SW2102.6 (COM)
- new net SW19: SW2034.6 (COM), SW2055.6 (COM), SW2072.6 (COM), SW2088.6 (COM)
- new net SW2: SW2001.6 (COM), SW2018.6 (COM), SW2038.6 (COM), SW2059.6 (COM), SW2075.6 (COM)
- new net SW20: SW2035.6 (COM), SW2056.6 (COM), SW2073.6 (COM), SW2089.6 (COM), SW2103.6 (COM)
- new net SW21: SW2036.6 (COM), SW2057.6 (COM), SW2090.6 (COM)
- new net SW3: SW2002.6 (COM), SW2019.6 (COM), SW2039.6 (COM), SW2060.6 (COM), SW2076.6 (COM), SW2093.6 (COM)
- new net SW4: SW2003.6 (COM), SW2020.6 (COM), SW2040.6 (COM), SW2061.6 (COM), SW2077.6 (COM)
- new net SW5: SW2004.6 (COM), SW2021.6 (COM), SW2041.6 (COM), SW2062.6 (COM), SW2078.6 (COM)
- new net SW6: SW2022.6 (COM), SW2042.6 (COM), SW2063.6 (COM), SW2079.6 (COM), SW2094.6 (COM)
- new net SW7: SW2005.6 (COM), SW2023.6 (COM), SW2043.6 (COM), SW2064.6 (COM), SW2080.6 (COM)
- new net SW8: SW2006.6 (COM), SW2024.6 (COM), SW2044.6 (COM), SW2065.6 (COM), SW2081.6 (COM)
- new net SW9: SW2007.6 (COM), SW2025.6 (COM), SW2045.6 (COM), SW2066.6 (COM), SW2082.6 (COM)
Other:
- moved on the sheet: SW2000B, SW2001B, SW2002B, SW2003B, SW2004B, SW2005B, SW2006B, SW2007B, SW2008B, SW2009B, SW2010B, SW2011B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
